File: PCB/0763-graviton.brd (EAGLE design)
At the start: 60 x 42 mm, 34 parts, among them J1 8-pin, J2 8-pin, J3 8-pin, J4 8-pin, SW1 MOM (OFF)-ON, SW2 MOM (OFF)-ON, U1 16-CH PWM Driver

Commit message: Graviton progress
Parts:
- R_REF: value (none) -> 600
Changed lines of the file:
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@@
 <?xml version="1.0" encoding="utf-8"?>
 <!DOCTYPE eagle SYSTEM "eagle.dtd">
-<eagle version="9.3.1">
+<eagle version="9.6.1">
 <drawing>
 <settings>
@@
 </layers>
 <board>
-<fusionsync huburn="a.cGVyc29uYWw6dWUyYmRlZGJl" projecturn="a.cGVyc29uYWw6dWUyYmRlZGJlIzIwMTgwNTA0MTMwNTkwMzU2" f3durn="urn:adsk.wipprod:dm.lineage:KwYG2HfnSrOsgiRrEmD8ow" pcbguid="bed4155a-2982-4baf-bcf1-5d4d607fec30" lastpulledtime="" lastsyncedchangeguid="4e1187b3-ce2f-06f1-0049-943fa142af90"/>
+<fusionsync huburn="a.cGVyc29uYWw6dWUyYmRlZGJl" projecturn="a.cGVyc29uYWw6dWUyYmRlZGJlIzIwMTgwNTA0MTMwNTkwMzU2" f3durn="urn:adsk.wipprod:dm.lineage:KwYG2HfnSrOsgiRrEmD8ow" pcbguid="bed4155a-2982-4baf-bcf1-5d4d607fec30" lastpulledtime="" lastsyncedchangeguid="4e1187b3-ce2f-06f1-0049-943fa142af90" latestrevisionid="" lastsyncedrevisionid="" lastboardhashguid="" lastpushedtime="" linktopcb3d="%12"/>
 <plain>
 <text x="7.3516" y="36.85" size="1.778" layer="21" ratio="15">0763A</text>
@@
 <attribute name="VALUE" x="5.475" y="10.16" size="0.4064" layer="27" font="vector" rot="R90" align="center"/>
 </element>
-<element name="R_REF" library="rlc" library_urn="urn:adsk.eagle:library:4192893" package="0603-RES" package3d_urn="urn:adsk.eagle:package:4193040/2" value="" x="27.0256" y="13.9192" smashed="yes" rot="MR0">
+<element name="R_REF" library="rlc" library_urn="urn:adsk.eagle:library:4192893" package="0603-RES" package3d_urn="urn:adsk.eagle:package:4193040/2" value="600" x="27.0256" y="13.9192" smashed="yes" rot="MR0">
 <attribute name="NAME" x="27.556" y="15.0876" size="0.8128" layer="26" font="vector" ratio="15" rot="MR0" align="center-left"/>
 <attribute name="VALUE" x="27.0256" y="13.9192" size="0.2" layer="28" rot="MR0" align="center"/>
